File: eagle/ovms_lilygo_tcall.brd (EAGLE design)
At the start: 98.1 x 49.5 mm, 45 parts, among them IC2 SN65HVD233, IC3 SN65HVD233, IC4 LMR516XX, IC5 MCP2515, Q1 X49SM16MSD2SC

Commit message: Correct width an hole position of case
Parts:
- R11: value 47k -> 470k
- R3: value 22k -> 220k
Changed lines of the file:
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@@
 <attribute name="VALUE" x="78.232" y="17.648" size="1.016" layer="28" ratio="10" rot="MR0"/>
 </element>
-<element name="R3" library="rcl" library_urn="urn:adsk.eagle:library:334" package="M0805" package3d_urn="urn:adsk.eagle:package:23556/2" value="22k" x="72.771" y="24.511" smashed="yes" rot="MR0">
+<element name="R3" library="rcl" library_urn="urn:adsk.eagle:library:334" package="M0805" package3d_urn="urn:adsk.eagle:package:23556/2" value="220k" x="72.771" y="24.511" smashed="yes" rot="MR0">
 <attribute name="NAME" x="70.231" y="23.876" size="1.27" layer="26" rot="MR0"/>
 <attribute name="POPULARITY" value="45" x="72.771" y="24.511" size="1.778" layer="28" rot="MR0" display="off"/>
@@
 <attribute name="VALUE" x="73.025" y="18.415" size="1.27" layer="28" rot="MR180"/>
 </element>
-<element name="R11" library="rcl" library_urn="urn:adsk.eagle:library:334" package="M0805" package3d_urn="urn:adsk.eagle:package:23556/2" value="47k" x="73.66" y="20.955" smashed="yes" rot="MR90">
+<element name="R11" library="rcl" library_urn="urn:adsk.eagle:library:334" package="M0805" package3d_urn="urn:adsk.eagle:package:23556/2" value="470k" x="73.66" y="20.955" smashed="yes" rot="MR90">
 <attribute name="NAME" x="74.295" y="17.78" size="1.27" layer="26" rot="MR0"/>
 <attribute name="POPULARITY" value="45" x="73.66" y="20.955" size="1.778" layer="28" rot="MR90" display="off"/>

Commit message: Clean up Eagle
Parts:
- C12: device rcl:C3216 -> rcl:C1206K
- R1: value 47k -> 470k
- R2: value 10k -> 100k
Changed lines of the file:
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@@
 <attribute name="VALUE" x="45.08" y="30.21" size="1.016" layer="28" rot="MR270"/>
 </element>
-<element name="R1" library="rcl" library_urn="urn:adsk.eagle:library:334" package="M0805" package3d_urn="urn:adsk.eagle:package:23556/2" value="47k" x="73.025" y="40.64" smashed="yes" rot="MR180">
+<element name="R1" library="rcl" library_urn="urn:adsk.eagle:library:334" package="M0805" package3d_urn="urn:adsk.eagle:package:23556/2" value="470k" x="73.025" y="40.64" smashed="yes" rot="MR180">
 <attribute name="NAME" x="75.311" y="41.021" size="1.27" layer="26" rot="MR180"/>
 <attribute name="POPULARITY" value="45" x="73.025" y="40.64" size="1.778" layer="28" rot="MR180" display="off"/>
@@
 <attribute name="VALUE" x="71.755" y="43.18" size="1.27" layer="28" rot="MR180"/>
 </element>
-<element name="R2" library="rcl" library_urn="urn:adsk.eagle:library:334" package="M0805" package3d_urn="urn:adsk.eagle:package:23556/2" value="10k" x="73.025" y="43.18" smashed="yes" rot="MR0">
+<element name="R2" library="rcl" library_urn="urn:adsk.eagle:library:334" package="M0805" package3d_urn="urn:adsk.eagle:package:23556/2" value="100k" x="73.025" y="43.18" smashed="yes" rot="MR0">
 <attribute name="NAME" x="77.851" y="42.545" size="1.27" layer="26" rot="MR0"/>
 <attribute name="POPULARITY" value="45" x="73.025" y="43.18" size="1.778" layer="28" rot="MR0" display="off"/>
@@
 <attribute name="VALUE" x="42.18" y="29.215" size="1.016" layer="27"/>
 </element>
-<element name="C12" library="rcl" library_urn="urn:adsk.eagle:library:334" package="C3216" package3d_urn="urn:adsk.eagle:package:23628/2" value="22u" x="49.784" y="43.18" smashed="yes" rot="MR90">
+<element name="C12" library="rcl" library_urn="urn:adsk.eagle:library:334" package="C1206K" package3d_urn="urn:adsk.eagle:package:23682/2" value="22u" x="49.784" y="43.18" smashed="yes" rot="MR90">
 <attribute name="NAME" x="51.054" y="46.355" size="1.27" layer="26" rot="MR0"/>
-<attribute name="POPULARITY" value="4" x="49.784" y="43.18" size="1.778" layer="28" rot="MR90" display="off"/>
+<attribute name="POPULARITY" value="13" x="49.784" y="43.18" size="1.778" layer="28" rot="MR90" display="off"/>
 <attribute name="SPICEPREFIX" value="C" x="49.784" y="43.18" size="1.778" layer="28" rot="MR90" display="off"/>
 <attribute name="VALUE" x="47.244" y="41.91" size="1.27" layer="28" rot="MR90"/>
@@
 <contactref element="C13" pad="+"/>
 <wire x1="45.63" y1="43.815" x2="47.535" y2="41.91" width="1.27" layer="16"/>
-<wire x1="49.654" y1="41.91" x2="49.784" y2="41.78" width="1.27" layer="16"/>
+<wire x1="49.654" y1="41.91" x2="49.784" y2="41.68" width="1.27" layer="16"/>
 <wire x1="47.535" y1="41.91" x2="49.654" y2="41.91" width="1.27" layer="16"/>
-<wire x1="49.784" y1="41.78" x2="49.914" y2="41.91" width="1.27" layer="16"/>
+<wire x1="49.784" y1="41.68" x2="49.914" y2="41.91" width="1.27" layer="16"/>
 <wire x1="49.914" y1="41.91" x2="53.975" y2="41.91" width="1.27" layer="16"/>
 <wire x1="49.48" y1="43.18" x2="50.165" y2="42.495" width="1.27" layer="1"/>

Commit message: Adjust resistors for low current (DCDC off)
Parts:
- R11: value 470k -> 220k
- R3: value 220k -> 100k
Changed lines of the file:
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@@
 <attribute name="VALUE" x="78.232" y="17.648" size="1.016" layer="28" ratio="10" rot="MR0"/>
 </element>
-<element name="R3" library="rcl" library_urn="urn:adsk.eagle:library:334" package="M0805" package3d_urn="urn:adsk.eagle:package:23556/2" value="220k" x="72.771" y="24.511" smashed="yes" rot="MR0">
+<element name="R3" library="rcl" library_urn="urn:adsk.eagle:library:334" package="M0805" package3d_urn="urn:adsk.eagle:package:23556/2" value="100k" x="72.771" y="24.511" smashed="yes" rot="MR0">
 <attribute name="NAME" x="70.231" y="23.876" size="1.27" layer="26" rot="MR0"/>
 <attribute name="POPULARITY" value="45" x="72.771" y="24.511" size="1.778" layer="28" rot="MR0" display="off"/>
@@
 <attribute name="VALUE" x="73.025" y="18.415" size="1.27" layer="28" rot="MR180"/>
 </element>
-<element name="R11" library="rcl" library_urn="urn:adsk.eagle:library:334" package="M0805" package3d_urn="urn:adsk.eagle:package:23556/2" value="470k" x="73.66" y="20.955" smashed="yes" rot="MR90">
+<element name="R11" library="rcl" library_urn="urn:adsk.eagle:library:334" package="M0805" package3d_urn="urn:adsk.eagle:package:23556/2" value="220k" x="73.66" y="20.955" smashed="yes" rot="MR90">
 <attribute name="NAME" x="74.295" y="17.78" size="1.27" layer="26" rot="MR0"/>
 <attribute name="POPULARITY" value="45" x="73.66" y="20.955" size="1.778" layer="28" rot="MR90" display="off"/>
