File: eagle/ovms_lilygo_tcall_revB.brd (EAGLE design)
At the start: 98.1 x 49.5 mm, 45 parts, among them IC2 SN65HVD233, IC3 SN65HVD233, IC4 LMR516XX, IC5 MCP2515, Q1 X49SM16MSD2SC

Commit message: Change schematic to increase default DCDC output voltage
Parts:
- R9: value 20k -> 18k
Changed lines of the file:
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@@
 <attribute name="VALUE" x="77.47" y="18.415" size="1.27" layer="28" rot="MR180"/>
 </element>
-<element name="R9" library="rcl" library_urn="urn:adsk.eagle:library:334" package="M0805" package3d_urn="urn:adsk.eagle:package:23556/2" value="20k" x="74.295" y="15.875" smashed="yes" rot="MR180">
+<element name="R9" library="rcl" library_urn="urn:adsk.eagle:library:334" package="M0805" package3d_urn="urn:adsk.eagle:package:23556/2" value="18k" x="74.295" y="15.875" smashed="yes" rot="MR180">
 <attribute name="NAME" x="73.025" y="14.605" size="1.27" layer="26" rot="MR180"/>
 <attribute name="POPULARITY" value="45" x="74.295" y="15.875" size="1.778" layer="28" rot="MR180" display="off"/>

Commit message: Replace CAN transceiver (TCAN330)
Parts:
- IC2, IC3: value SN65HVD233 -> TCAN330DR
Changed lines of the file:
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@@
 </element>
 <element name="LILYGO" library="ovms_lilygo" package="LILYGO-TCALL-A7670E_1.0" value="LILYGO-T-CALL-A7670E_1.0SIMCOMTOP" x="57.15" y="22.86" smashed="yes"/>
-<element name="IC2" library="ovms_lilygo" package="SO-08" value="SN65HVD233" x="36.83" y="28.575" smashed="yes" rot="MR270">
+<element name="IC2" library="ovms_lilygo" package="SO-08" value="TCAN330DR" x="36.83" y="28.575" smashed="yes" rot="MR270">
 <attribute name="NAME" x="35.56" y="25.908" size="1.27" layer="26" rot="MR180"/>
 <attribute name="VALUE" x="38.735" y="24.638" size="1.27" layer="28" rot="MR0"/>
 </element>
-<element name="IC3" library="ovms_lilygo" package="SO-08" value="SN65HVD233" x="30.48" y="19.05" smashed="yes" rot="MR270">
+<element name="IC3" library="ovms_lilygo" package="SO-08" value="TCAN330DR" x="30.48" y="19.05" smashed="yes" rot="MR270">
 <attribute name="NAME" x="31.75" y="14.732" size="1.27" layer="26" rot="MR0"/>
 <attribute name="VALUE" x="32.385" y="15.113" size="1.27" layer="28" rot="MR0"/>
